File: KiCad-Files/MotorSpeedControl.kicad_pcb (KiCad board)
At the start: 2 copper layers, 84 x 84 mm, 25 parts, among them J1 Throttle, J2 AC IN, J3 Motor, J4 Tachometer, Q1 NTPF190N65S3H, SW1 SW_Push, U1 RAC10E-12SK, U2 RAC10E-12SK, U3 ADuM4120

Commit message: Updated schematic.
Parts:
- added R3: 100k, Resistors_SMD:R_0805, F.Cu at (105.8, 58.2)
- added R4: 470k 0.25W, Resistors_ThroughHole:R_Axial_DIN0207_L6.3mm_D2.5mm_P7.62mm_Horizontal, B.Cu at (149.0, 123.0)
Routing:
- net GND: track 174.9 -> 179.8 mm
- net Net-(A1-Pad19): track 36.2 -> 38.9 mm
